File: line/line.kicad_pcb (KiCad board)
At the start: 2 copper layers, 75 x 75 mm, 41 parts, among them J1 MAINS, J2 CONTROL, Q1 Q_NMOS_GDS, Q2 Q_NMOS_GDS, U1 LM324, U2 LTV-817S

Commit message: WIP
Parts:
- added H1: MountingHole, MountingHole:MountingHole_3.7mm_Pad_Via, F.Cu at (105.0, 137.0)
- added H2: MountingHole, MountingHole:MountingHole_3.7mm_Pad_Via, F.Cu at (155.0, 137.0)
- D3, D4, D5, D6, D7, D8: value BAT54W -> SS13A; footprint Package_TO_SOT_SMD:SOT-323_SC-70 -> Diode_SMD:D_SMA_Handsoldering
- J1: footprint Drake:HB-9500-3P -> Drake:HB-9500-4P
- NT1: footprint NetTie:NetTie-2_THT_Pad0.3mm -> NetTie:NetTie-2_SMD_Pad0.5mm
- Q1, Q2: value Q_NMOS_GDS -> WMM38N60C2
- R14: value 270??? -> 3R9
- TP1, TP2, TP3, TP4, TP5, TP6, TP7, TP8: footprint TestPoint:TestPoint_Pad_D3.0mm -> TestPoint:TestPoint_Pad_D2.0mm
- moved J1 52.5 mm to (115.8, 132.8)
- moved R1 49.6 mm to (107.0, 130.0), turned to 180 degrees
- moved C1 42.1 mm to (113.0, 123.0), turned to -90 degrees
- moved C3 36.5 mm to (117.0, 125.0), turned to -90 degrees
- moved J2 33.6 mm to (153.5, 118.5), turned to 90 degrees
- moved NT1 33.4 mm to (130.0, 93.5), turned to -90 degrees
- moved C2 32.4 mm to (117.0, 113.0), turned to -90 degrees
- moved TP3 29.4 mm to (110.0, 106.0)
- moved TP1 29.3 mm to (105.0, 106.0)
- moved R9 28.9 mm to (158.0, 125.0), turned to -90 degrees
- moved Q1 26.7 mm to (150.0, 90.0)
- moved U2 26.1 mm to (150.0, 125.0), turned to 180 degrees
- moved R2 24.7 mm to (113.0, 113.0), turned to 90 degrees
- moved D1 23.7 mm to (105.0, 123.0), turned to -90 degrees
- moved R8 23.7 mm to (140.0, 125.0), turned to 180 degrees
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Connections:
- D3 pad 1: Net-(D1-K) -> VCC
- D3 pad 2: unconnected-(D3-NC-Pad2) -> Net-(D1-K)
- D4 pad 1: Net-(D4-A) -> GND
- D4 pad 2: unconnected-(D4-NC-Pad2) -> Net-(D4-A)
- D5 pad 1: Net-(D5-A) -> Net-(D5-K)
- D5 pad 2: unconnected-(D5-NC-Pad2) -> Net-(D5-A)
- D6 pad 1: Net-(D6-A) -> Net-(D6-K)
- D6 pad 2: unconnected-(D6-NC-Pad2) -> Net-(D6-A)
- D7 pad 1: GND -> Net-(D5-A)
- D7 pad 2: unconnected-(D7-NC-Pad2) -> GND
- D8 pad 1: GND -> Net-(D6-A)
- D8 pad 2: unconnected-(D8-NC-Pad2) -> GND
- J1 pad 2: /MAINS_L_IN -> /MAINS_N
- J1 pad 3: /MAINS_L_OUT -> /MAINS_L_IN
Routing:
- net /MAINS_L_IN: track 0.00 -> 38.4 mm
- net /MAINS_L_OUT: track 0.00 -> 32.1 mm
- net Net-(Q1-G): track 0.00 -> 26.8 mm, vias 0 -> 2
- net /S2S: track 0.00 -> 26.8 mm
- added copper zone on B.Cu, net /MAINS_L_IN
- added copper zone on F.Cu, net /MAINS_L_IN
- added copper zone on B.Cu, net /MAINS_L_OUT
- added copper zone on F.Cu, net /MAINS_L_OUT
- added copper zone on B.Cu, net GND
- added copper zone on F.Cu, net GND
Other:
- board size 75 x 75 mm -> 60 x 80 mm

Commit message: WIP
Parts:
- removed NT1: NetTie_2, NetTie:NetTie-2_SMD_Pad0.5mm
- moved Q1 10.5 mm to (142.7, 82.5)
- moved Q2 7.75 mm to (117.3, 92.5)
Connections:
- J1 pad 1: /MAINS_N -> /MAINS_L_IN
- J1 pad 3: /MAINS_L_IN -> /MAINS_N
- Q1 pad 3: /S2S -> GND
- Q2 pad 3: /S2S -> GND
Routing:
- net /MAINS_L_IN: track 38.4 -> 0.00 mm, vias 0 -> 60
- net /MAINS_L_OUT: track 32.1 -> 0.00 mm, vias 0 -> 57
- net Net-(Q1-G): track 26.8 -> 0.00 mm, vias 2 -> 0
- net /S2S: track 26.8 -> 0.00 mm
- added copper zone on B.Cu, net /MAINS_N

Commit message: WIP
Parts:
- added TP9: GND, TestPoint:TestPoint_Pad_D2.0mm, F.Cu at (137.0, 73.0)
- moved D1 37.0 mm to (105.0, 86.0)
- moved D2 37.0 mm to (105.0, 76.0)
- moved D3 37.0 mm to (110.0, 86.0)
- moved D4 37.0 mm to (110.0, 76.0)
- moved R1 36.0 mm to (107.0, 94.0)
- moved TP8 35.1 mm to (143.0, 73.0)
- moved TP6 35.0 mm to (149.0, 73.0)
- moved TP7 35.0 mm to (155.0, 73.0)
- moved R10 34.1 mm to (138.0, 91.0), turned to 90 degrees
- moved C1 34.0 mm to (114.0, 89.0)
- moved R2 34.0 mm to (114.0, 79.0)
- moved R8 34.0 mm to (141.0, 91.0), turned to -90 degrees
- moved C2 34.0 mm to (117.0, 79.0)
- moved C3 34.0 mm to (117.0, 91.0)
- moved C4 34.0 mm to (144.0, 80.0)
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Routing:
- net VCC: track 0.00 -> 83.9 mm, vias 0 -> 3
- net Net-(D1-K): track 0.00 -> 62.4 mm, vias 0 -> 3
- net /MAINS_N: track 0.00 -> 58.2 mm, vias 0 -> 1
- net Net-(U1C-+): track 0.00 -> 42.1 mm, vias 0 -> 3
- net Net-(Q1-G): track 0.00 -> 40.1 mm, vias 0 -> 2
- net Net-(D4-A): track 0.00 -> 39.6 mm
- net Net-(R14-Pad1): track 0.00 -> 32.9 mm, vias 0 -> 2
- net Net-(D6-A): track 0.00 -> 31.4 mm, vias 0 -> 2
- net Net-(U1D--): track 0.00 -> 30.0 mm
- net Net-(D5-A): track 0.00 -> 25.9 mm
- net Net-(D5-K): track 0.00 -> 25.2 mm
- net Net-(U1D-+): track 0.00 -> 23.9 mm
- net Net-(D6-K): track 0.00 -> 18.8 mm
- net GND: track 0.00 -> 15.0 mm, vias 0 -> 49
- net Net-(J2-Pin_2): track 0.00 -> 12.4 mm
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- added copper zone on F.Cu, net /MAINS_N

Commit message: WIP
Parts:
- J2: value CONTROL -> PWM
Other:
- board text added: "+"
- board text added: "-"
- board text added: "230V 20A max."
- board text added: "3-5V"
- board text added: "L-IN"
- board text added: "L-OUT"
- board text added: "N-IN"
- board text added: "N-OUT"
- board text added: "drake.cz"
- board text added: "powreg v1.0"

Commit message: WIP
Parts:
- D1: value BYG10J (J/K/M/Y) -> ES1J
- D2: value SMAZ20-13-F -> 1SMA4747A

Commit message: WIP
Parts:
- removed the D4 at (110.0, 76.0)
- removed D7, D8: SS13A, Diode_SMD:D_SMA_Handsoldering
- removed the R1 at (107.0, 94.0)
- removed the R10 at (138.0, 91.0)
- removed R13: 1M, Resistor_SMD:R_0805_2012Metric_Pad1.20x1.40mm_HandSolder
- removed the R4 at (117.0, 85.0)
- removed the R6 at (129.0, 91.0)
- removed the R7 at (144.0, 85.0)
- removed the R8 at (141.0, 91.0)
- removed the TP4 at (129.0, 73.0)
- removed the TP5 at (129.0, 85.0)
- removed the U1 at (137.0, 83.0)
- added C2: 10u/50V, Capacitor_SMD:C_1206_3216Metric_Pad1.33x1.80mm_HandSolder, F.Cu at (64.8, 83.1)
- added C6: 10u/50V, Capacitor_SMD:C_1206_3216Metric_Pad1.33x1.80mm_HandSolder, F.Cu at (64.8, 86.5)
- added C7: 10u/50V, Capacitor_SMD:C_1206_3216Metric_Pad1.33x1.80mm_HandSolder, F.Cu at (64.8, 89.8)
- added D5: 1SMA4747A, Diode_SMD:D_SMA, F.Cu at (57.8, 84.9)
- added R11: 100k (250mW min.), Resistor_SMD:R_1206_3216Metric_Pad1.30x1.75mm_HandSolder, F.Cu at (70.8, 86.3)
- added R12: 100k (250mW min.), Resistor_SMD:R_1206_3216Metric_Pad1.30x1.75mm_HandSolder, F.Cu at (70.8, 89.6)
- added R2: 100k (250mW min.), Resistor_SMD:R_1206_3216Metric_Pad1.30x1.75mm_HandSolder, F.Cu at (70.8, 79.7)
- added R3: 100k (250mW min.), Resistor_SMD:R_1206_3216Metric_Pad1.30x1.75mm_HandSolder, F.Cu at (70.8, 83.0)
- added R9: 270R, Resistor_SMD:R_0805_2012Metric_Pad1.20x1.40mm_HandSolder, F.Cu at (76.1, 82.5)
- added U2: LM358, Package_SO:SOIC-8_3.9x4.9mm_P1.27mm, F.Cu at (74.5, 100.1)
- added U3: TLP2345, Package_SO:SO-6L_10x3.84mm_P1.27mm, F.Cu at (68.0, 94.2)
- C1: value 10u/25V -> 10u/50V; footprint Capacitor_SMD:C_0805_2012Metric_Pad1.18x1.45mm_HandSolder -> Capacitor_SMD:C_1206_3216Metric_Pad1.33x1.80mm_HandSolder
- D1: value ES1J -> AB10S-DC; footprint Diode_SMD:D_SMA_Handsoldering -> Diode_SMD:Diode_Bridge_Diotec_ABS
- D2, D3: footprint Diode_SMD:D_SMA_Handsoldering -> Diode_SMD:D_SMA
- D4: renamed from D5; footprint Diode_SMD:D_SMA_Handsoldering -> Diode_SMD:D_SMA
- D6: value SS13A -> ES1D; footprint Diode_SMD:D_SMA_Handsoldering -> Diode_SMD:D_SMA
- R1: renamed from R9; value 270 -> 270R
- R5: value 1M -> 220k
- moved D6 65.4 mm to (57.8, 89.5)
- moved R5 52.9 mm to (76.1, 79.6), turned to 0 degrees
- moved D3 52.5 mm to (57.8, 80.4), turned to 0 degrees
- moved C1 50.1 mm to (64.8, 79.8), turned to 0 degrees
- moved D1 41.4 mm to (66.0, 100.1), turned to 0 degrees
- moved C3 41.2 mm to (76.2, 85.5), turned to 0 degrees
- moved D4 32.0 mm to (91.0, 72.0)
- moved D2 14.3 mm to (91.0, 79.0)
- renumbered C2 to C4, C4 to C5, J2 to J1, J1 to J2, R14 to R10, R2 to R4, R3 to R6, R11 to R7, R12 to R8, TP3 to TP2, TP2 to TP3, TP9 to TP4, TP6 to TP5, TP7 to TP6, TP8 to TP7, U2 to U1
Connections:
- C3 pad 1: Net-(D6-A) -> VCC
- C4 pad 1: Net-(D5-A) -> Net-(D4-A)
- D1 pad 2: Net-(D1-A) -> GND
- D4 pad 2: Net-(D5-A) -> Net-(D4-A)
- Q1 pad 2: /MAINS_L_OUT -> /MAINS_L_IN
- Q1 pad 3: GND -> Net-(D5-A)
- Q2 pad 2: /MAINS_L_IN -> /MAINS_L_OUT
- Q2 pad 3: GND -> Net-(D5-A)
- R10 pad 1: Net-(R14-Pad1) -> Net-(U3-VO)
- R4 pad 1: VCC -> Net-(U2A--)
- R4 pad 2: Net-(D4-A) -> VCC
- R5 pad 1: Net-(D5-A) -> GND
- R5 pad 2: Net-(U1C-+) -> Net-(U2A--)
- R6 pad 2: Net-(D5-A) -> Net-(D4-A)
- TP2 pad 1: Net-(D4-A) -> Net-(U2A--)
- TP5 pad 1: Net-(U1D--) -> Net-(D4-A)
- TP7 pad 1: Net-(R14-Pad1) -> Net-(R9-Pad1)
Routing:
- net (no net): track 0.00 -> 52.9 mm
- net Net-(D1-+): track 62.4 -> 14.2 mm, vias 3 -> 0
- net Net-(U1C-+): track 42.1 -> 0.00 mm, vias 3 -> 0
- net Net-(D4-A): track 39.6 -> 0.00 mm
- net VCC: track 83.9 -> 50.2 mm, vias 3 -> 0
- net Net-(R14-Pad1): track 32.9 -> 0.00 mm, vias 2 -> 0
- net Net-(U1D--): track 30.0 -> 0.00 mm
- net Net-(D5-A): track 25.9 -> 0.00 mm
- net Net-(D6-A): track 31.4 -> 6.00 mm, vias 2 -> 0
- net Net-(D4-K): track 25.2 -> 0.00 mm
- net Net-(U2B-+): track 23.9 -> 0.00 mm
- net Net-(D5-K): track 18.8 -> 0.00 mm
- net Net-(J1-Pin_2): track 12.4 -> 0.00 mm
- net Net-(U1C--): track 9.59 -> 0.00 mm
- net Net-(R10-Pad1): track 8.20 -> 0.00 mm
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Other:
- board text added: "powreg v1.1"
- board text removed: "powreg v1.0"
