File: line/line.kicad_sch (KiCad schematic)
At the start: 41 parts, among them J1 MAINS, J2 CONTROL, Q1 Q_NMOS_GDS, Q2 Q_NMOS_GDS, U1 LM324, U2 LTV-817S

Commit message: WIP
Parts:
- added H1, H2: MountingHole, MountingHole:MountingHole_3.7mm_Pad_Via, symbol Mechanical:MountingHole
- D3, D4, D5, D6, D7, D8: value BAT54W -> SS13A; footprint Package_TO_SOT_SMD:SOT-323_SC-70 -> Diode_SMD:D_SMA_Handsoldering; symbol Diode:BAT54W -> Device:D_Schottky
- J1: footprint Drake:HB-9500-3P -> Drake:HB-9500-4P; symbol Connector_Generic:Conn_01x03 -> Connector_Generic:Conn_01x04
- NT1: footprint NetTie:NetTie-2_THT_Pad0.3mm -> NetTie:NetTie-2_SMD_Pad0.5mm
- Q1, Q2: value Q_NMOS_GDS -> WMM38N60C2
- R14: value 270??? -> 3R9
- TP1, TP2, TP3, TP4, TP5, TP6, TP7, TP8: footprint TestPoint:TestPoint_Pad_D3.0mm -> TestPoint:TestPoint_Pad_D2.0mm
Connections:
- net GND: now also D4.1 (K), D7.2 (A), D8.2 (A); no longer D4.3 (K), D7.1 (A), D8.1 (A)
- net MAINS_L_IN: now also J1.3 (Pin_3); no longer J1.2 (Pin_2)
- net MAINS_L_OUT: now also J1.4 (Pin_4); no longer J1.3 (Pin_3)
- net MAINS_N: now also J1.2 (Pin_2)
- net VCC: now also D3.1 (K); no longer D3.3 (K)
- net at C2.1, R3.2, R5.1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: now also D5.2 (A), D7.1 (K); no longer D5.1 (A), D7.3 (K)
- net at R3.1, U1.1: now also D5.1 (K); no longer D5.3 (K)
- net at R2.2, TP3.1, U1.2 (-)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: now also D4.2 (A); no longer D4.1 (A)
- net at C3.1, R4.2, R6.1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: now also D6.2 (A), D8.1 (K); no longer D6.1 (A), D8.3 (K)
- net at D1.1 (K), D2.1 (K), TP1.1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: now also D3.2 (A); no longer D3.1 (A)
- net at R4.1, U1.7: now also D6.1 (K); no longer D6.3 (K)

Commit message: WIP
Parts:
- removed NT1: NetTie_2, NetTie:NetTie-2_SMD_Pad0.5mm, symbol Device:NetTie_2
Connections:
- net S2S is gone; now on net GND: Q1.3 (S), Q2.3 (S)
- net MAINS_L_IN: now also J1.1 (Pin_1); no longer J1.3 (Pin_3)
- net MAINS_N: now also J1.3 (Pin_3); no longer J1.1 (Pin_1)
Changed lines of the file:
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@@
     (effects (font (size 1.27 1.27)) (justify right bottom))
   )
-  (label "MAINS_L_IN" (at 85.09 121.92 0) (fields_autoplaced)
+  (label "MAINS_L_IN" (at 85.09 127 0) (fields_autoplaced)
     (effects (font (size 1.27 1.27)) (justify left bottom))
   )
@@
     (effects (font (size 1.27 1.27)) (justify left bottom))
   )
-  (label "S2S" (at 251.46 71.12 180) (fields_autoplaced)
-    (effects (font (size 0.8 0.8) (color 72 72 72 1)) (justify right bottom))
-  )
   (label "MAINS_N" (at 85.09 124.46 0) (fields_autoplaced)
     (effects (font (size 1.27 1.27)) (justify left bottom))
   )
-  (label "MAINS_N" (at 85.09 127 0) (fields_autoplaced)
+  (label "MAINS_N" (at 85.09 121.92 0) (fields_autoplaced)
     (effects (font (size 1.27 1.27)) (justify left bottom))
   )
@@
     )
   )
-  (symbol (lib_id "power:GND") (at 259.08 71.12 90) (unit 1)
+  (symbol (lib_id "power:GND") (at 254 71.12 90) (unit 1)
     (in_bom yes) (on_board yes) (dnp no) (fields_autoplaced)
-    (property "Reference" "#PWR015" (at 265.43 71.12 0)
+    (property "Reference" "#PWR015" (at 260.35 71.12 0)
       (effects (font (size 1.27 1.27)) hide)
     )
-    (property "Value" "GND" (at 262.255 71.4368 90)
+    (property "Value" "GND" (at 257.175 71.4368 90)
       (effects (font (size 1.27 1.27)) (justify right))
     )
-    (property "Footprint" "" (at 259.08 71.12 0)
+    (property "Footprint" "" (at 254 71.12 0)
       (effects (font (size 1.27 1.27)) hide)
     )
-    (property "Datasheet" "" (at 259.08 71.12 0)
+    (property "Datasheet" "" (at 254 71.12 0)
       (effects (font (size 1.27 1.27)) hide)
     )
@@
         )
       )
-    )
-  )
-  (symbol (lib_id "Device:NetTie_2") (at 256.54 71.12 0) (unit 1)
-    (in_bom no) (on_board yes) (dnp no) (fields_autoplaced)
-    (property "Reference" "NT1" (at 256.54 70.0311 0)
-      (effects (font (size 1.27 1.27)))
-    )
-    (property "Value" "NetTie_2" (at 256.54 70.0311 0)
-      (effects (font (size 1.27 1.27)) hide)
-    )
-    (property "Footprint" "NetTie:NetTie-2_SMD_Pad0.5mm" (at 256.54 71.12 0)
-      (effects (font (size 1.27 1.27)) hide)
-    )
-    (property "Datasheet" "~" (at 256.54 71.12 0)
-      (effects (font (size 1.27 1.27)) hide)
-    )
-    (pin "1")
-    (pin "2")
-    (instances
-      (project "line"
-        (path "/2b625d23-24b6-4053-9c0b-d9a46cc4ab31"
-          (reference "NT1") (unit 1)
-        )
-      )

Commit message: WIP
Parts:
- added TP9: GND, TestPoint:TestPoint_Pad_D2.0mm, symbol Connector:TestPoint
Connections:
- net GND: now also TP9.1
Changed lines of the file:
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@@
+    )
+  )
+  (symbol (lib_id "Connector:TestPoint") (at 106.68 118.11 0) (unit 1)
+    (in_bom yes) (on_board yes) (dnp no)
+    (property "Reference" "TP9" (at 106.68 109.22 0)
+      (effects (font (size 1.27 1.27)))
+    )
+    (property "Value" "GND" (at 106.68 111.76 0)
+      (effects (font (size 1.27 1.27)))
+    )
+    (property "Footprint" "TestPoint:TestPoint_Pad_D2.0mm" (at 111.76 118.11 0)
+      (effects (font (size 1.27 1.27)) hide)
+    )
+    (property "Datasheet" "~" (at 111.76 118.11 0)
+      (effects (font (size 1.27 1.27)) hide)
+    )
+    (pin "1")
+    (instances
+      (project "line"
+        (path "/2b625d23-24b6-4053-9c0b-d9a46cc4ab31"
+          (reference "TP9") (unit 1)
+        )
+      )
     )
   )
@@
         )
       )
+    )
+  )
+  (symbol (lib_id "power:GND") (at 106.68 118.11 0) (unit 1)
+    (in_bom yes) (on_board yes) (dnp no) (fields_autoplaced)
+    (property "Reference" "#PWR016" (at 106.68 124.46 0)
+      (effects (font (size 1.27 1.27)) hide)
+    )
+    (property "Value" "GND" (at 106.68 122.2455 0)
+      (effects (font (size 1.27 1.27)))
+    )
+    (property "Footprint" "" (at 106.68 118.11 0)
+      (effects (font (size 1.27 1.27)) hide)
+    )
+    (property "Datasheet" "" (at 106.68 118.11 0)
+      (effects (font (size 1.27 1.27)) hide)
+    )
+    (pin "1")
+    (instances
+      (project "line"
+        (path "/2b625d23-24b6-4053-9c0b-d9a46cc4ab31"
+          (reference "#PWR016") (unit 1)
+        )
+      )

Commit message: WIP
Parts:
- J2: value CONTROL -> PWM
Changed lines of the file:
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@@
       (effects (font (size 1.27 1.27)))
     )
-    (property "Value" "CONTROL" (at 179.07 113.2111 0)
+    (property "Value" "PWM" (at 179.07 113.2111 0)
       (effects (font (size 1.27 1.27)))
     )

Commit message: WIP
Parts:
- D1: value BYG10J (J/K/M/Y) -> ES1J
- D2: value SMAZ20-13-F -> 1SMA4747A
Changed lines of the file:
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@@
-(kicad_sch (version 20230221) (generator eeschema)
+(kicad_sch (version 20230409) (generator eeschema)
   (paper "A4")
   (junction (at 130.81 66.04) (diameter 0) (color 0 0 0 0)
@@
     (stroke (width 0) (type default))
   )
-  (text "https://tinyurl.com/2y7xszn5" (at 177.8 162.56 0)
+  (text "https://tinyurl.com/2y7xszn5" (exclude_from_sim no)
+ (at 177.8 162.56 0)
     (effects (font (size 1.27 1.27)) (justify left bottom))
   )
@@
       (effects (font (size 1.27 1.27)) (justify left))
     )
-    (property "Value" "SMAZ20-13-F" (at 59.182 83.8273 90)
+    (property "Value" "1SMA4747A" (at 59.182 83.8273 90)
       (effects (font (size 1.27 1.27)) (justify left))
     )
@@
       (effects (font (size 1.27 1.27)) hide)
     )
-    (property "Datasheet" "https://www.tme.eu/Document/834adb1f38dda1a8a8e74929a7ec261d/SMAZx-13-F.pdf" (at 57.15 82.55 0)
+    (property "Datasheet" "https://datasheet.lcsc.com/lcsc/1912111437_LGE-1SMA4747A_C362318.pdf" (at 57.15 82.55 0)
       (effects (font (size 1.27 1.27)) hide)
     )
@@
       (effects (font (size 1.27 1.27)))
     )
-    (property "Value" "BYG10J (J/K/M/Y)" (at 49.53 61.1411 0)
-      (effects (font (size 1.27 1.27)))
-    )
+    (property "Value" "ES1J" (at 49.53 61.1411 0)
+      (effects (font (size 1.27 1.27)))
+    )

Commit message: WIP
Parts:
- removed D1: ES1J, Diode_SMD:D_SMA_Handsoldering, symbol Device:D
- removed D4, D6, D7, D8: SS13A, Diode_SMD:D_SMA_Handsoldering, symbol Device:D_Schottky
- removed R1: 100k (250mW min.), Resistor_SMD:R_1206_3216Metric_Pad1.30x1.75mm_HandSolder, symbol Device:R
- removed R10: 20k, Resistor_SMD:R_0805_2012Metric_Pad1.20x1.40mm_HandSolder, symbol Device:R
- removed R13, R6: 1M, Resistor_SMD:R_0805_2012Metric_Pad1.20x1.40mm_HandSolder, symbol Device:R
- removed R4: 220k, Resistor_SMD:R_0805_2012Metric_Pad1.20x1.40mm_HandSolder, symbol Device:R
- removed R7: 82k, Resistor_SMD:R_0805_2012Metric_Pad1.20x1.40mm_HandSolder, symbol Device:R
- removed R8: 100k, Resistor_SMD:R_0805_2012Metric_Pad1.20x1.40mm_HandSolder, symbol Device:R
- removed TP4: SAW+, TestPoint:TestPoint_Pad_D2.0mm, symbol Connector:TestPoint
- removed TP5: SAW-, TestPoint:TestPoint_Pad_D2.0mm, symbol Connector:TestPoint
- removed U1: LM324, Package_SO:SOIC-14_3.9x8.7mm_P1.27mm, symbol Amplifier_Operational:LM324
- added C2, C6, C7: 10u/50V, Capacitor_SMD:C_1206_3216Metric_Pad1.33x1.80mm_HandSolder, symbol Device:C
- added C8: 100n, Capacitor_SMD:C_0805_2012Metric_Pad1.18x1.45mm_HandSolder, symbol Device:C
- added D1: AB10S-DC, Diode_SMD:Diode_Bridge_Diotec_ABS, symbol Diode_Bridge:ABS10
- added D5: 1SMA4747A, Diode_SMD:D_SMA, symbol Device:D_Zener
- added D6: ES1D, Diode_SMD:D_SMA, symbol Diode:US1D
- added R11, R12, R2, R3: 100k (250mW min.), Resistor_SMD:R_1206_3216Metric_Pad1.30x1.75mm_HandSolder, symbol Device:R
- added R9: 270R, Resistor_SMD:R_0805_2012Metric_Pad1.20x1.40mm_HandSolder, symbol Device:R
- added TP10: OG, TestPoint:TestPoint_Pad_D2.0mm, symbol Connector:TestPoint
- added TP8: O+, TestPoint:TestPoint_Pad_D2.0mm, symbol Connector:TestPoint
- added TP9: O-, TestPoint:TestPoint_Pad_D2.0mm, symbol Connector:TestPoint
- added U2: LM358, Package_SO:SOIC-8_3.9x4.9mm_P1.27mm, symbol Amplifier_Operational:LM358
- added U3: TLP2345, Package_SO:SO-6L_10x3.84mm_P1.27mm, symbol Isolator:TLP2761
- C1: value 10u/25V -> 10u/50V; footprint Capacitor_SMD:C_0805_2012Metric_Pad1.18x1.45mm_HandSolder -> Capacitor_SMD:C_1206_3216Metric_Pad1.33x1.80mm_HandSolder
- D2, D3: footprint Diode_SMD:D_SMA_Handsoldering -> Diode_SMD:D_SMA
- D4: renamed from D5; footprint Diode_SMD:D_SMA_Handsoldering -> Diode_SMD:D_SMA
- R1: renamed from R9; value 270 -> 270R
- R5: value 1M -> 220k
- renumbered C2 to C4, C4 to C5, J2 to J1, J1 to J2, R14 to R10, R2 to R4, R3 to R6, R11 to R7, R12 to R8, TP3 to TP2, TP2 to TP3, TP9 to TP4, TP6 to TP5, TP7 to TP6, TP8 to TP7, U2 to U1
Connections:
- net GND: now also R5.1, C2.2, D1.2 (-), U2.4 (V-), U3.3 (K); no longer Q1.3 (S), Q2.3 (S)
- net MAINS_L_IN: now also Q1.2 (D), R2.2, R3.2; no longer Q2.2 (D)
- net MAINS_L_OUT: now also Q2.2 (D); no longer Q1.2 (D)
- net MAINS_N: now also D1.3, R11.1, R12.1
- net VCC: now also C3.1, R4.2, C2.1, U2.8 (V+); no longer R4.1
- net at D4.1 (K), R6.1: now also U2.1
- net at C4.1, D4.2 (A), R6.2: now also TP5.1, U2.6 (-); no longer R5.1
- net at TP2.1: now also R4.1, R5.2, U2.2 (-); no longer R4.2
- net at R10.1: now also U3.5 (VO); no longer TP7.1
- net at Q1.1 (G), Q2.1 (G), R10.2: now also TP10.1
- net at D2.1 (K), D3.2 (A), TP1.1: now also D1.1 (+), U2.3 (+)
- net at C5.1, R7.1, R8.2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: now also U2.5 (+)
- new net: C6.1, C7.1, C8.1, D5.1 (K), D6.1 (K), TP8.1, U3.6 (VDD)
- new net: C6.2, C7.2, C8.2, D5.2 (A), Q1.3 (S), Q2.3 (S), TP9.1, U3.4 (GND)
- new net: D1.4, R2.1, R3.1
- new net: D6.2 (A), R11.2, R12.2
- new net: R9.1, TP7.1, U2.7
- new net: R9.2, U3.1 (A)
Other:
- note added: "https://tinyurl.com/2drzcton"
- note removed: "https://tinyurl.com/2y7xszn5"
- moved on the sheet: C4, C5, D2, D4, H1, H2, J1, J2, Q1, Q2, R1, R10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

Commit message: WIP
Parts:
- added R13: 56k, Resistor_SMD:R_0805_2012Metric_Pad1.20x1.40mm_HandSolder, symbol Device:R
- R3: value 100k (250mW min.) -> 100k/250mW
Connections:
- net MAINS_L_IN: now also D1.4; no longer R2.2, R3.2
- net at U1.3: now also R13.2; no longer R7.2
- net at D2.1 (K), TP1.1, U2.3 (+): now also R3.1; no longer D1.1 (+), D3.2 (A)
- new net: R13.1, R7.2
- new net: D1.1 (+), R3.2
- now unconnected: R2.1
Other:
- moved on the sheet: R2, R3
Changed lines of the file:
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@@
   (junction (at 237.49 147.32) (diameter 0) (color 0 0 0 0)
   )
-  (junction (at 72.39 73.66) (diameter 0) (color 0 0 0 0)
-  )
   (junction (at 158.75 102.87) (diameter 0) (color 0 0 0 0)
   )
@@
   (junction (at 175.26 48.26) (diameter 0) (color 0 0 0 0)
   )
-  (junction (at 104.14 100.33) (diameter 0) (color 0 0 0 0)
-  )
   (junction (at 158.75 96.52) (diameter 0) (color 0 0 0 0)
-  )
-  (junction (at 72.39 81.28) (diameter 0) (color 0 0 0 0)
   )
   (junction (at 237.49 115.57) (diameter 0) (color 0 0 0 0)
@@
     (stroke (width 0) (type default))
   )
+  (wire (pts (xy 80.01 100.33) (xy 85.09 100.33))
+    (stroke (width 0) (type default))
+  )
   (wire (pts (xy 175.26 48.26) (xy 175.26 46.99))
     (stroke (width 0) (type default))
   )
-  (wire (pts (xy 62.23 38.1) (xy 156.21 38.1))
-    (stroke (width 0) (type default))
-  )
   (wire (pts (xy 228.6 105.41) (xy 231.14 105.41))
     (stroke (width 0) (type default))
@@
     (stroke (width 0) (type default))
   )
-  (wire (pts (xy 104.14 100.33) (xy 125.73 100.33))
-    (stroke (width 0) (type default))
-  )
   (wire (pts (xy 158.75 113.03) (xy 158.75 115.57))
     (stroke (width 0) (type default))
@@
     (stroke (width 0) (type default))
   )
-  (wire (pts (xy 72.39 63.5) (xy 72.39 73.66))
+  (wire (pts (xy 72.39 63.5) (xy 72.39 92.71))
     (stroke (width 0) (type default))
   )
@@
     (stroke (width 0) (type default))
   )
+  (wire (pts (xy 92.71 100.33) (xy 96.52 100.33))
+    (stroke (width 0) (type default))
+  )
+  (wire (pts (xy 62.23 38.1) (xy 148.59 38.1))
+    (stroke (width 0) (type default))
+  )
   (wire (pts (xy 248.92 63.5) (xy 266.7 63.5))
     (stroke (width 0) (type default))
@@
     (stroke (width 0) (type default))
   )
-  (wire (pts (xy 80.01 100.33) (xy 96.52 100.33))
-    (stroke (width 0) (type default))
-  )
   (wire (pts (xy 242.57 95.25) (xy 247.65 95.25))
     (stroke (width 0) (type default))
@@
     (stroke (width 0) (type default))
   )
-  (wire (pts (xy 72.39 73.66) (xy 74.93 73.66))
+  (wire (pts (xy 34.29 120.65) (xy 39.37 120.65))
     (stroke (width 0) (type default))
   )
@@
     (stroke (width 0) (type dash) (color 255 0 0 1))
   )
-  (wire (pts (xy 96.52 100.33) (xy 104.14 100.33))
+  (wire (pts (xy 96.52 100.33) (xy 125.73 100.33))
     (stroke (width 0) (type default))
   )
@@
     (stroke (width 0) (type default))
   )
-  (wire (pts (xy 104.14 72.39) (xy 104.14 100.33))
-    (stroke (width 0) (type default))
-  )
   (wire (pts (xy 242.57 95.25) (xy 242.57 101.6))
     (stroke (width 0) (type default))
@@
     (stroke (width 0) (type default))
   )
-  (wire (pts (xy 72.39 81.28) (xy 74.93 81.28))
+  (wire (pts (xy 34.29 128.27) (xy 39.37 128.27))
     (stroke (width 0) (type default))
   )
@@
     (stroke (width 0) (type default))
   )
-  (wire (pts (xy 72.39 81.28) (xy 72.39 92.71))
-    (stroke (width 0) (type default))
-  )
   (wire (pts (xy 120.65 105.41) (xy 120.65 107.95))
     (stroke (width 0) (type default))
   )
   (wire (pts (xy 237.49 63.5) (xy 238.76 63.5))
-    (stroke (width 0) (type default))
-  )
-  (wire (pts (xy 69.85 73.66) (xy 72.39 73.66))
-    (stroke (width 0) (type default))
-  )
-  (wire (pts (xy 69.85 81.28) (xy 72.39 81.28))
     (stroke (width 0) (type default))
   )
@@
     )
   )
-  (symbol (lib_id "Device:R") (at 69.85 77.47 180) (unit 1)
+  (symbol (lib_id "Device:R") (at 34.29 124.46 180) (unit 1)
     (in_bom yes) (on_board yes) (dnp no)
-    (property "Reference" "R2" (at 77.47 73.66 0)
+    (property "Reference" "R2" (at 41.91 120.65 0)
       (effects (font (size 1.27 1.27)) (justify right))
     )
-    (property "Value" "100k (250mW min.)" (at 72.39 78.74 0)
+    (property "Value" "100k (250mW min.)" (at 36.83 125.73 0)
       (effects (font (size 1.27 1.27)) (justify right) hide)
     )
-    (property "Footprint" "Resistor_SMD:R_1206_3216Metric_Pad1.30x1.75mm_HandSolder" (at 71.628 77.47 90)
-      (effects (font (size 1.27 1.27)) hide)
-    )
-    (property "Datasheet" "~" (at 69.85 77.47 0)
+    (property "Footprint" "Resistor_SMD:R_1206_3216Metric_Pad1.30x1.75mm_HandSolder" (at 36.068 124.46 90)
+      (effects (font (size 1.27 1.27)) hide)
+    )
+    (property "Datasheet" "~" (at 34.29 124.46 0)
       (effects (font (size 1.27 1.27)) hide)
     )
@@
     )
   )
-  (symbol (lib_id "Device:R") (at 74.93 77.47 180) (unit 1)
+  (symbol (lib_id "Device:R") (at 88.9 100.33 270) (unit 1)
     (in_bom yes) (on_board yes) (dnp no)
-    (property "Reference" "R3" (at 77.47 76.2 0)
+    (property "Reference" "R3" (at 90.17 102.87 90)
       (effects (font (size 1.27 1.27)) (justify right))
     )
-    (property "Value" "100k (250mW min.)" (at 77.47 78.74 0)
+    (property "Value" "100k/250mW" (at 95.25 105.41 90)
       (effects (font (size 1.27 1.27)) (justify right))
     )
-    (property "Footprint" "Resistor_SMD:R_1206_3216Metric_Pad1.30x1.75mm_HandSolder" (at 76.708 77.47 90)
-      (effects (font (size 1.27 1.27)) hide)
-    )
-    (property "Datasheet" "~" (at 74.93 77.47 0)
+    (property "Footprint" "Resistor_SMD:R_1206_3216Metric_Pad1.30x1.75mm_HandSolder" (at 88.9 98.552 90)
+      (effects (font (size 1.27 1.27)) hide)
+    )
+    (property "Datasheet" "~" (at 88.9 100.33 0)
       (effects (font (size 1.27 1.27)) hide)
     )
@@
         )
       )
+    )
+  )
+  (symbol (lib_id "Device:R") (at 152.4 38.1 270) (unit 1)
+    (in_bom yes) (on_board yes) (dnp no) (fields_autoplaced)
+    (property "Reference" "R13" (at 152.4 34.0741 90)
+      (effects (font (size 1.27 1.27)))
+    )
+    (property "Value" "56k" (at 152.4 35.9951 90)
+      (effects (font (size 1.27 1.27)))
+    )
+    (property "Footprint" "Resistor_SMD:R_0805_2012Metric_Pad1.20x1.40mm_HandSolder" (at 152.4 36.322 90)
+      (effects (font (size 1.27 1.27)) hide)
+    )
+    (property "Datasheet" "~" (at 152.4 38.1 0)
+      (effects (font (size 1.27 1.27)) hide)
+    )
+    (pin "1")
+    (pin "2")
+    (instances
+      (project "line"
+        (path "/2b625d23-24b6-4053-9c0b-d9a46cc4ab31"
+          (reference "R13") (unit 1)
+        )
+      )

Commit message: WIP
Parts:
- removed C1: 10u/50V, Capacitor_SMD:C_1206_3216Metric_Pad1.33x1.80mm_HandSolder, symbol Device:C
- removed D3: SS13A, Diode_SMD:D_SMA, symbol Device:D_Schottky
- removed U2: LM358, Package_SO:SOIC-8_3.9x4.9mm_P1.27mm, symbol Amplifier_Operational:LM358
- added C10, C11, C12, C13, C9: 100n/500V, Capacitor_SMD:C_1210_3225Metric_Pad1.33x2.70mm_HandSolder, symbol Device:C
- added C14: 100n, Capacitor_SMD:C_0805_2012Metric_Pad1.18x1.45mm_HandSolder, symbol Device:C
- added D7: SS13A, Diode_SMD:D_SMA, symbol Device:D_Schottky
- added D8: 1SMA4747A, Diode_SMD:D_SMA, symbol Device:D_Zener
- added R14: 100R, Resistor_SMD:R_1206_3216Metric_Pad1.30x1.75mm_HandSolder, symbol Device:R
- added R15: 1M, Resistor_SMD:R_0805_2012Metric_Pad1.20x1.40mm_HandSolder, symbol Device:R
- added TP11: SAW+, TestPoint:TestPoint_Pad_D2.0mm, symbol Connector:TestPoint
- added U5: LM324, symbol Amplifier_Operational:LM324
- C2: value 10u/50V -> 100u/25V
- R11, R12: value 100k (250mW min.) -> 100k
- R2: value 100k (250mW min.) -> 1M
- R3: value 100k/250mW -> 1M
- R4: value 1M -> 220k
- R5: value 220k -> 1M
- TP2: value THD -> SAW+
- TP5: value SAW -> SAW+
Connections:
- net GND: now also C14.2, D8.2 (A), U5.11 (V-), U5.2 (-), U5.5 (+); no longer R5.1
- net MAINS_L_IN: now also R2.2, R3.2, C10.1, C11.1, C12.1, C13.1, C9.1; no longer D1.4
- net MAINS_N: now also R14.1; no longer D1.3
- net VCC: now also D1.1 (+), D8.1 (K), U5.4 (V+); no longer R4.2
- net at D4.1 (K), R6.1: now also U5.1
- net at C4.1, D4.2 (A), R6.2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: now also R5.2
- net at R2.1: now also D1.4, C10.2, C11.2, C12.2, C13.2, C9.2
- net at D2.1 (K), R3.1, TP1.1: now also U5.3 (+), U5.6 (-)
- net at R9.1, TP7.1: now also U5.8
- net at C5.1, R7.1, R8.2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: now also U5.10 (+)
- new net: C14.1, D7.2 (A), R15.2, R4.2, TP2.1
- new net: R15.1, R5.1, TP11.1, U5.9 (-)
- new net: D1.3, R14.2
- new net: D7.1 (K), R4.1, U5.7
Other:
- note added: "https://tinyurl.com/2gpgmr7y"
- note removed: "https://tinyurl.com/2drzcton"
- moved on the sheet: C2, C3, C4, D1, D2, D4, R6, TP1, TP5
